Commit message: Add lopsided sub

File: catkin_ws/src/aquadrone_description/models/v2_wobbly.urdf.xacro (robot description, xacro)
@@ -8,5 +8,5 @@
   <xacro:include filename="$(find aquadrone_description)/urdf/thruster.urdf.xacro"/>
   <!-- Create the rov_example -->
-  <xacro:aquadrone_base debug="$(arg debug)" cog="0 0 0" cob="0 0 0"/>
+  <xacro:aquadrone_base debug="$(arg debug)" cog="0.02 0.02 0" cob="-0.02 -0.02 0"/>
     <!-- Pressure  -->
   <xacro:include filename="$(find uuv_sensor_ros_plugins)/urdf/pressure_snippets.xacro"/>

File: catkin_ws/src/aquadrone_description/urdf/aquadrone_v2.urdf.xacro (robot description, xacro)
@@ -15,8 +15,4 @@
 -->
   <!-- https://github.com/uuvsimulator/uuv_simulator/wiki/Templates-to-create-a-new-thruster-actuated-vehicle-model -->
-  <!-- Center of gravity -->
-  <xacro:property name="cog" value="0 0 0"/>
-  <!-- Center of buoyancy -->
-  <xacro:property name="cob" value="0 0 0"/>
   <!-- Fluid density -->
   <xacro:property name="rho" value="1028"/>
@@ -28,5 +24,5 @@
   <xacro:property name="mass" value="${width * length * height * rho}"/>
   <!-- Vehicle macro -->
-  <xacro:macro name="aquadrone_base" params="debug">
+  <xacro:macro name="aquadrone_base" params="debug cog cob">
     <!-- Rigid body description of the base link -->
     <link name="base_link">
