Commit message: Sim model now has 2 thrusters

File: catkin_ws/src/aquadrone_description/models/v2.urdf.xacro (robot description, xacro)
@@ -7,3 +7,9 @@
   <!-- Create the rov_example -->
   <xacro:aquadrone_base debug="$(arg debug)"/>
+  <xacro:thruster_macro thruster_id="0">
+    <origin xyz="0 0.5 0" rpy="0 0 0"/>
+  </xacro:thruster_macro>
+  <xacro:thruster_macro thruster_id="1">
+    <origin xyz="0 -0.5 0" rpy="0 0 0"/>
+  </xacro:thruster_macro>
 </robot>

File: catkin_ws/src/aquadrone_description/urdf/aquadrone_v2.urdf.xacro (robot description, xacro)
@@ -1,10 +1,18 @@
 <?xml version="1.0"?>
 <robot xmlns:xacro="http://www.ros.org/wiki/xacro">
+<!-- ORIGINAL SOURCE OF FILES - Modified for UW Aquadrone
+     Copyright (c) 2016 The UUV Simulator Authors.
+     All rights reserved.
+     Licensed under the Apache License, Version 2.0 (the "License");
+     you may not use this file except in compliance with the License.
+     You may obtain a copy of the License at
+       http://www.apache.org/licenses/LICENSE-2.0
+     Unless required by applicable law or agreed to in writing, software
+     distributed under the License is distributed on an "AS IS" BASIS,
+     WITHOUT WARRANTIES OR CONDITIONS OF ANY KIND, either express or implied.
+     See the License for the specific language governing permissions and
+     limitations under the License.
+-->
   <!-- https://github.com/uuvsimulator/uuv_simulator/wiki/Templates-to-create-a-new-thruster-actuated-vehicle-model -->
-  <!--
-    Vehicle's parameters
-  -->
-  <xacro:property name="mass" value="60"/>
-  <xacro:property name="volume" value="0.1"/>
   <!-- Center of gravity -->
   <xacro:property name="cog" value="0 0 0"/>
@@ -17,4 +25,6 @@
   <xacro:property name="width"  value="0.3048"/>
   <xacro:property name="height" value="0.2"/>
+  <xacro:property name="volume" value="${width * length * height}"/>
+  <xacro:property name="mass" value="${width * length * height * rho}"/>
   <!-- Vehicle macro -->
   <xacro:macro name="aquadrone_base" params="debug">
@@ -47,23 +57,17 @@
     <gazebo>
       <plugin name="uuv_plugin" filename="libuuv_underwater_object_plugin.so">
-        <!-- Fluid density to be used in the computation of buoyancy forces
-        for all links specified below -->
         <fluid_density>${rho}</fluid_density>
-        <!-- Name of the current velocity topic -->
         <flow_velocity_topic>hydrodynamics/current_velocity</flow_velocity_topic>
-        <!-- Debug flag, if set to true, added-mass, damping and restoring
-        forces and moments will be published in separate topics -->
         <debug>${debug}</debug>
-        <!-- List of hydrodynamic models this robot's links -->
         <link name="base_link">
           <!-- This flag will make the link neutrally buoyant -->
-          <neutrally_buoyant>1</neutrally_buoyant>
-          <!-- Center of buoyancy -->
+          <neutrally_buoyant>0</neutrally_buoyant>
           <center_of_buoyancy>${cob}</center_of_buoyancy>
-          <!--
-          Reference:
-          Fossen, Thor I. Handbook of marine craft hydrodynamics and motion
-          control. John Wiley & Sons, 2011.
-          -->
+          <volume>${volume*1.005}</volume>
+          <box>
+            <width>${width}</width>
+            <length>${length}</length>
+            <height>${height}</height>
+          </box>
           <!-- Fossen's equation of motion -->
           <hydrodynamic_model>
@@ -82,5 +86,5 @@
             -->
             <linear_damping>
-              -1 -1 -1 0 0 0
+              -3 -3 -3 -1 -1 -1
             </linear_damping>
             <!--
@@ -100,13 +104,7 @@
               0 0 0 0 0 0
             </quadratic_damping>
-                      <!-- Link's bounding box, it is used to recalculate the immersed
+          <!-- Link's bounding box, it is used to recalculate the immersed
           volume when close to the surface.
           This is a workaround the invalid bounding box given by Gazebo-->
-          <volume>${width * length * height}</volume>
-          <box>
-            <width>${width}</width>
-            <length>${length}</length>
-            <height>${height}</height>
-          </box>
           </hydrodynamic_model>
         </link>
@@ -114,3 +112,51 @@
     </gazebo>
   </xacro:macro>
+  <xacro:macro name="thruster_macro" params="thruster_id *origin">
+    <link name="thruster_${thruster_id}">
+      <visual>
+        <geometry>
+          <box size="0.01 0.01 0.1"/>
+        </geometry>
+      </visual>
+      <inertial>
+        <mass value="0.001" />
+        <origin xyz="0 0 0" rpy="0 0 0"/>
+        <inertia ixx="0.000000017" ixy="0.0" ixz="0.0"
+               iyy="0.000000017" iyz="0.0"
+               izz="0.000000017" />
+      </inertial>
+    </link>
+    <!-- Joint between thruster link and vehicle base link -->
+    <joint name="thruster_${thruster_id}_joint" type="continuous">
+      <xacro:insert_block name="origin" />
+      <axis xyz="1 0 0" />
+      <parent link="base_link" />
+      <child link="thruster_${thruster_id}" />
+    </joint>
+    <gazebo>
+      <!-- Thruster ROS plugin -->
+      <plugin name="${thruster_id}_thruster_model" filename="libuuv_thruster_ros_plugin.so">
+        <thrusterID>${thruster_id}</thrusterID>
+        <linkName>thruster_${thruster_id}</linkName>
+        <jointName>thruster_${thruster_id}_joint</jointName>
+        <thrustTopic>thrusters/${thruster_id}/thrust</thrustTopic>
+        <inputTopic>thrusters/${thruster_id}/input</inputTopic>
+        <gain>1</gain>
+        <clampMax>1</clampMax>
+        <clampMin>-1</clampMin>
+        <thrust_efficiency>1</thrust_efficiency>
+        <propeller_efficiency>1</propeller_efficiency>
+        <dynamics>
+          <type>ZeroOrder</type>
+        </dynamics>
+        <conversion>
+          <type>Basic</type>
+          <rotorConstant>1.0</rotorConstant>
+        </conversion>
+      </plugin>
+    </gazebo>
+    <gazebo reference="thruster_${thruster_id}">
+      <selfCollide>false</selfCollide>
+    </gazebo>
+  </xacro:macro>
 </robot>

Commit message: Model has 6 thrusters, pressure sensor, and imu

File: catkin_ws/src/aquadrone_description/models/v2.urdf.xacro (robot description, xacro)
@@ -5,11 +5,34 @@
   <!-- Include the ROV macro file -->
   <xacro:include filename="$(find aquadrone_description)/urdf/aquadrone_v2.urdf.xacro"/>
+  <xacro:include filename="$(find aquadrone_description)/urdf/thruster.urdf.xacro"/>
   <!-- Create the rov_example -->
   <xacro:aquadrone_base debug="$(arg debug)"/>
+    <!-- Pressure  -->
+  <xacro:include filename="$(find uuv_sensor_ros_plugins)/urdf/pressure_snippets.xacro"/>
+  <xacro:default_pressure namespace="aquadrone_v2/out/" parent_link="base_link">
+    <origin xyz="0 0 0" rpy="0 0 0"/>
+  </xacro:default_pressure>
+  <!-- IMU -->
+  <xacro:include filename="$(find uuv_sensor_ros_plugins)/urdf/imu_snippets.xacro"/>
+  <xacro:default_imu namespace="aquadrone_v2/out/" parent_link="base_link">
+    <origin xyz="0 0 0" rpy="0 0 0"/>
+  </xacro:default_imu>
   <xacro:thruster_macro thruster_id="0">
-    <origin xyz="0 0.5 0" rpy="0 0 0"/>
+    <origin xyz="0.4 0.4 0" rpy="0 ${pi/4} ${pi/2}"/>
   </xacro:thruster_macro>
   <xacro:thruster_macro thruster_id="1">
-    <origin xyz="0 -0.5 0" rpy="0 0 0"/>
+    <origin xyz="0.4 -0.4 0" rpy="0 ${pi/4} ${-pi/2}"/>
+  </xacro:thruster_macro>
+  <xacro:thruster_macro thruster_id="2">
+    <origin xyz="0 0.4 0" rpy="0 0 0"/>
+  </xacro:thruster_macro>
+  <xacro:thruster_macro thruster_id="3">
+    <origin xyz="0 -0.4 0" rpy="0 0 0"/>
+  </xacro:thruster_macro>
+  <xacro:thruster_macro thruster_id="4">
+    <origin xyz="-0.4 0.4 0" rpy="0 ${-pi/4} ${pi/2}"/>
+  </xacro:thruster_macro>
+  <xacro:thruster_macro thruster_id="5">
+    <origin xyz="-0.4 -0.4 0" rpy="0 ${-pi/4} ${-pi/2}"/>
   </xacro:thruster_macro>
 </robot>

File: catkin_ws/src/aquadrone_description/urdf/aquadrone_v2.urdf.xacro (robot description, xacro)
@@ -42,4 +42,10 @@
         <geometry>
           <box size="${length} ${width} ${height}"/>
+        </geometry>
+      </visual>
+      <visual>
+        <origin xyz="${length/2} 0 0" rpy="0 0 0"/>
+        <geometry>
+          <sphere radius="${width/2}"/>
         </geometry>
       </visual>
@@ -112,51 +118,3 @@
     </gazebo>
   </xacro:macro>
-  <xacro:macro name="thruster_macro" params="thruster_id *origin">
-    <link name="thruster_${thruster_id}">
-      <visual>
-        <geometry>
-          <box size="0.01 0.01 0.1"/>
-        </geometry>
-      </visual>
-      <inertial>
-        <mass value="0.001" />
-        <origin xyz="0 0 0" rpy="0 0 0"/>
-        <inertia ixx="0.000000017" ixy="0.0" ixz="0.0"
-               iyy="0.000000017" iyz="0.0"
-               izz="0.000000017" />
-      </inertial>
-    </link>
-    <!-- Joint between thruster link and vehicle base link -->
-    <joint name="thruster_${thruster_id}_joint" type="continuous">
-      <xacro:insert_block name="origin" />
-      <axis xyz="1 0 0" />
-      <parent link="base_link" />
-      <child link="thruster_${thruster_id}" />
-    </joint>
-    <gazebo>
-      <!-- Thruster ROS plugin -->
-      <plugin name="${thruster_id}_thruster_model" filename="libuuv_thruster_ros_plugin.so">
-        <thrusterID>${thruster_id}</thrusterID>
-        <linkName>thruster_${thruster_id}</linkName>
-        <jointName>thruster_${thruster_id}_joint</jointName>
-        <thrustTopic>thrusters/${thruster_id}/thrust</thrustTopic>
-        <inputTopic>thrusters/${thruster_id}/input</inputTopic>
-        <gain>1</gain>
-        <clampMax>1</clampMax>
-        <clampMin>-1</clampMin>
-        <thrust_efficiency>1</thrust_efficiency>
-        <propeller_efficiency>1</propeller_efficiency>
-        <dynamics>
-          <type>ZeroOrder</type>
-        </dynamics>
-        <conversion>
-          <type>Basic</type>
-          <rotorConstant>1.0</rotorConstant>
-        </conversion>
-      </plugin>
-    </gazebo>
-    <gazebo reference="thruster_${thruster_id}">
-      <selfCollide>false</selfCollide>
-    </gazebo>
-  </xacro:macro>
 </robot>

Commit message: Get first version of sim thruster control working. Work to improve organization

File: catkin_ws/src/aquadrone_description/models/v2.urdf.xacro (robot description, xacro)
@@ -32,8 +32,8 @@
   </xacro:thruster_macro>
   <xacro:thruster_macro thruster_id="4">
-    <origin xyz="-0.4 0.4 0" rpy="0 ${-pi/4} ${pi/2}"/>
+    <origin xyz="-0.4 0.4 0" rpy="0 ${pi/4} ${pi/2}"/>
   </xacro:thruster_macro>
   <xacro:thruster_macro thruster_id="5">
-    <origin xyz="-0.4 -0.4 0" rpy="0 ${-pi/4} ${-pi/2}"/>
+    <origin xyz="-0.4 -0.4 0" rpy="0 ${pi/4} ${-pi/2}"/>
   </xacro:thruster_macro>
 </robot>
