Commit message: Created and quickly tested -thruster configuration

File: catkin_ws/src/aquadrone_description/models/v28.urdf.xacro (robot description, xacro)
@@ -8,5 +8,5 @@
   <xacro:include filename="$(find aquadrone_description)/urdf/thruster.urdf.xacro"/>
   <!-- Create the rov_example -->
-  <xacro:aquadrone_base debug="$(arg debug)" cog="0.0000001 0.0000001 0" cob="-0.0000001 -0.0000001 0"/>
+  <xacro:aquadrone_base debug="$(arg debug)" cog="0 0 0" cob="0 0 0"/>
     <!-- Pressure  -->
   <xacro:include filename="$(find uuv_sensor_ros_plugins)/urdf/pressure_snippets.xacro"/>
@@ -20,20 +20,26 @@
   </xacro:default_imu>
   <xacro:thruster_macro thruster_id="0">
-    <origin xyz="0.4 0.4 0" rpy="0 ${pi/4} ${pi/2}"/>
+    <origin xyz="0.4 0.4 -0.2" rpy="0 ${pi/2} 0"/>
   </xacro:thruster_macro>
   <xacro:thruster_macro thruster_id="1">
-    <origin xyz="0.4 -0.4 0" rpy="0 ${pi/4} ${-pi/2}"/>
+    <origin xyz="0.4 -0.4 -0.2" rpy="0 ${pi/2} 0"/>
   </xacro:thruster_macro>
   <xacro:thruster_macro thruster_id="2">
+    <origin xyz="-0.4 0.4 -0.2" rpy="0 ${pi/2} 0"/>
+  </xacro:thruster_macro>
+  <xacro:thruster_macro thruster_id="3">
+    <origin xyz="-0.4 -0.4 -0.2" rpy="0 ${pi/2} 0"/>
+  </xacro:thruster_macro>
+ <xacro:thruster_macro thruster_id="4">
     <origin xyz="0 0.4 0" rpy="0 0 0"/>
   </xacro:thruster_macro>
-  <xacro:thruster_macro thruster_id="3">
+   <xacro:thruster_macro thruster_id="5">
     <origin xyz="0 -0.4 0" rpy="0 0 0"/>
   </xacro:thruster_macro>
-  <xacro:thruster_macro thruster_id="4">
-    <origin xyz="-0.4 0.4 0" rpy="0 ${-pi/4} ${pi/2}"/>
+<xacro:thruster_macro thruster_id="6">
+    <origin xyz="0.4 0 0.2" rpy="0 0 ${-pi/2}"/>
   </xacro:thruster_macro>
-  <xacro:thruster_macro thruster_id="5">
-    <origin xyz="-0.4 -0.4 0" rpy="0 ${-pi/4} ${-pi/2}"/>
+   <xacro:thruster_macro thruster_id="7">
+    <origin xyz="-0.4 0 0.2" rpy="0 0 ${-pi/2}"/>
   </xacro:thruster_macro>
 </robot>

Commit message: Add sensor module and simple simulated camera

File: catkin_ws/src/aquadrone_description/models/v28.urdf.xacro (robot description, xacro)
@@ -19,4 +19,8 @@
     <origin xyz="0 0 0" rpy="0 0 0"/>
   </xacro:default_imu>
+  <xacro:include filename="$(find aquadrone_description)/urdf/simple_camera.urdf.xacro"/>
+  <xacro:simple_camera_macro name="front_cam">
+    <origin xyz="0.5 0 0.2" rpy="0 0 0"/>
+  </xacro:simple_camera_macro>
   <!-- UP/DOWN-->
   <xacro:thruster_macro thruster_id="0">
