Commit message: Somewhat-working pole-finding demo. Needs debugging

File: catkin_ws/src/aquadrone_description/urdf/aquadrone_v2.urdf.xacro (robot description, xacro)
@@ -30,6 +30,6 @@
         <mass value="${mass}" />
         <origin xyz="${cog}" rpy="0 0 0"/>
-        <inertia ixx="1" ixy="0" ixz="0"
-                 iyy="1" iyz="0"
+        <inertia ixx="100" ixy="0" ixz="0"
+                 iyy="100" iyz="0"
                  izz="1" />
       </inertial>
@@ -104,5 +104,5 @@
             -->
             <quadratic_damping>
-              0 0 0 0 0 0
+              -1 -1 -1 -1 -1 -1
             </quadratic_damping>
           <!-- Link's bounding box, it is used to recalculate the immersed

File: catkin_ws/src/aquadrone_sim_worlds/demo_objects/blue_pole.urdf.xacro (robot description, xacro)
@@ -9,5 +9,5 @@
       <origin xyz="0 0 0"/>
       <geometry>
-        <cylinder radius="0.1" length="10" />
+        <cylinder radius="0.1" length="20" />
       </geometry>
     </visual>
@@ -15,5 +15,5 @@
       <origin xyz="0 0 0"/>
       <geometry>
-        <cylinder radius="0.1" length="10" />
+        <cylinder radius="0.1" length="20" />
       </geometry>
     </collision>

File: catkin_ws/src/aquadrone_sim_worlds/demo_objects/green_pole.urdf.xacro (robot description, xacro)
@@ -9,5 +9,5 @@
       <origin xyz="0 0 0"/>
       <geometry>
-        <cylinder radius="0.1" length="10" />
+        <cylinder radius="0.1" length="20" />
       </geometry>
     </visual>
@@ -15,5 +15,5 @@
       <origin xyz="0 0 0"/>
       <geometry>
-        <cylinder radius="0.1" length="10" />
+        <cylinder radius="0.1" length="20" />
       </geometry>
     </collision>

File: catkin_ws/src/aquadrone_sim_worlds/demo_objects/red_pole.urdf.xacro (robot description, xacro)
@@ -9,5 +9,5 @@
       <origin xyz="0 0 0"/>
       <geometry>
-        <cylinder radius="0.1" length="10" />
+        <cylinder radius="0.1" length="20" />
       </geometry>
     </visual>
@@ -15,5 +15,5 @@
       <origin xyz="0 0 0"/>
       <geometry>
-        <cylinder radius="0.1" length="10" />
+        <cylinder radius="0.1" length="20" />
       </geometry>
     </collision>

File: catkin_ws/src/aquadrone_sim_worlds/demo_objects/white_pole.urdf.xacro (robot description, xacro)
@@ -9,5 +9,5 @@
       <origin xyz="0 0 0"/>
       <geometry>
-        <cylinder radius="0.1" length="10" />
+        <cylinder radius="0.1" length="20" />
       </geometry>
     </visual>
@@ -15,5 +15,5 @@
       <origin xyz="0 0 0"/>
       <geometry>
-        <cylinder radius="0.1" length="10" />
+        <cylinder radius="0.1" length="20" />
       </geometry>
     </collision>
