Commit message: Just touch up model for sideways movement at the moment

File: aquadrone_description/models/v28.urdf.xacro (robot description, xacro)
@@ -45,8 +45,8 @@
 <!-- LEFT/RIGHT-->
 <xacro:thruster_macro thruster_id="6">
-    <origin xyz="0.4 0 0.2" rpy="0 0 ${-pi/2}"/>
+    <origin xyz="0.4 0 0.05" rpy="0 0 ${-pi/2}"/>
   </xacro:thruster_macro>
    <xacro:thruster_macro thruster_id="7">
-    <origin xyz="-0.4 0 0.2" rpy="0 0 ${-pi/2}"/>
+    <origin xyz="-0.4 0 0.05" rpy="0 0 ${-pi/2}"/>
   </xacro:thruster_macro>
 </robot>

Commit message: Update V2 model with CAD

File: aquadrone_description/models/v28.urdf.xacro (robot description, xacro)
@@ -4,4 +4,9 @@
   <!-- Input debug flag -->
   <xacro:arg name="debug" default="0"/>
+    <xacro:property name="strut_thickness" value="0.02"/>
+  <!-- Describing the dimensions of the vehicle's bounding box -->
+  <xacro:property name="length" value="0.51"/>
+  <xacro:property name="width"  value="0.46"/>
+  <xacro:property name="height" value="0.2"/>
   <!-- Include the ROV macro file -->
   <xacro:include filename="$(find aquadrone_description)/urdf/aquadrone_v2.urdf.xacro"/>
@@ -12,5 +17,5 @@
   <xacro:include filename="$(find uuv_sensor_ros_plugins)/urdf/pressure_snippets.xacro"/>
   <xacro:default_pressure namespace="aquadrone/out/" parent_link="base_link">
-    <origin xyz="0 0 0" rpy="0 0 0"/>
+        <origin xyz="0 0 ${0.11 + 0.2/2.0}" rpy="0 ${pi/2.0} 0"/>
   </xacro:default_pressure>
   <!-- IMU -->
@@ -21,32 +26,32 @@
   <xacro:include filename="$(find aquadrone_description)/urdf/simple_camera.urdf.xacro"/>
   <xacro:simple_camera_macro name="front_cam">
-    <origin xyz="0.5 0 0.2" rpy="0 0 0"/>
+    <origin xyz="${0.91/2.0 - 0.08 - 0.22/2.0} 0 ${0.11 + 0.2/2.0}" rpy="0 0 0"/>
   </xacro:simple_camera_macro>
   <!-- UP/DOWN-->
   <xacro:thruster_macro thruster_id="0">
-    <origin xyz="0.4 0.4 -0.2" rpy="0 ${pi/2} 0"/>
+    <origin xyz="0.2 0.285 0.1" rpy="0 ${pi/2} 0"/>
   </xacro:thruster_macro>
   <xacro:thruster_macro thruster_id="1">
-    <origin xyz="0.4 -0.4 -0.2" rpy="0 ${pi/2} 0"/>
+    <origin xyz="0.2 -0.285 0.1" rpy="0 ${pi/2} 0"/>
   </xacro:thruster_macro>
   <xacro:thruster_macro thruster_id="2">
-    <origin xyz="-0.4 0.4 -0.2" rpy="0 ${pi/2} 0"/>
+    <origin xyz="-0.2 0.285 0.1" rpy="0 ${pi/2} 0"/>
   </xacro:thruster_macro>
   <xacro:thruster_macro thruster_id="3">
-    <origin xyz="-0.4 -0.4 -0.2" rpy="0 ${pi/2} 0"/>
+    <origin xyz="-0.2 -0.285 0.1" rpy="0 ${pi/2} 0"/>
   </xacro:thruster_macro>
 <!-- FORWARD/BACKWARD-->
  <xacro:thruster_macro thruster_id="4">
-    <origin xyz="0 0.4 0" rpy="0 0 0"/>
+    <origin xyz="0 0.285 0.1" rpy="0 0 0"/>
   </xacro:thruster_macro>
    <xacro:thruster_macro thruster_id="5">
-    <origin xyz="0 -0.4 0" rpy="0 0 0"/>
+    <origin xyz="0 -0.285 0.1" rpy="0 0 0"/>
   </xacro:thruster_macro>
 <!-- LEFT/RIGHT-->
 <xacro:thruster_macro thruster_id="6">
-    <origin xyz="0.4 0 0.05" rpy="0 0 ${-pi/2}"/>
+    <origin xyz="0 0.17 0" rpy="0 0 ${-pi/2}"/>
   </xacro:thruster_macro>
    <xacro:thruster_macro thruster_id="7">
-    <origin xyz="-0.4 0 0.05" rpy="0 0 ${-pi/2}"/>
+    <origin xyz="0 -0.17 0" rpy="0 0 ${-pi/2}"/>
   </xacro:thruster_macro>
 </robot>

File: aquadrone_description/urdf/aquadrone_v2.urdf.xacro (robot description, xacro)
@@ -41,8 +41,4 @@
   <!-- Fluid density -->
   <xacro:property name="rho" value="1028"/>
-  <!-- Describing the dimensions of the vehicle's bounding box -->
-  <xacro:property name="length" value="0.9144"/>
-  <xacro:property name="width"  value="0.3048"/>
-  <xacro:property name="height" value="0.2"/>
   <xacro:property name="displaced_volume" value="${0.02074192626}"/>
   <xacro:property name="bouyancy_fudge_factor" value="1.08"/>
@@ -60,14 +56,55 @@
                  izz="4004" />
       </inertial>
+      <!-- Top Plate -->
       <visual>
-        <origin xyz="0 0 0" rpy="0 0 0"/>
+        <origin xyz="0 0 ${(height - strut_thickness)/2.0}" rpy="0 0 0"/>
         <geometry>
-          <box size="${length} ${width} ${height}"/>
+          <box size="${length} ${width} ${strut_thickness}"/>
+        </geometry>
+      </visual>
+      <!-- Bottom Plate -->
+      <visual>
+        <origin xyz="0 0 ${-(height - strut_thickness)/2.0}" rpy="0 0 0"/>
+        <geometry>
+          <box size="${length} ${width} 0.02"/>
+        </geometry>
+      </visual>
+      <!-- Verticals -->
+      <visual>
+        <origin xyz="${(length - strut_thickness)/2.0} ${(width - strut_thickness)/2.0} 0" rpy="0 0 0"/>
+        <geometry>
+          <box size="${strut_thickness} ${strut_thickness} ${height}"/>
         </geometry>
       </visual>
       <visual>
-        <origin xyz="${length/2} 0 0" rpy="0 0 0"/>
+        <origin xyz="${-(length - strut_thickness)/2.0} ${(width - strut_thickness)/2.0} 0" rpy="0 0 0"/>
         <geometry>
-          <sphere radius="${width/2}"/>
+          <box size="${strut_thickness} ${strut_thickness} ${height}"/>
+        </geometry>
+      </visual>
+      <visual>
+        <origin xyz="${(length - strut_thickness)/2.0} ${-(width - strut_thickness)/2.0} 0" rpy="0 0 0"/>
+        <geometry>
+          <box size="${strut_thickness} ${strut_thickness} ${height}"/>
+        </geometry>
+      </visual>
+      <visual>
+        <origin xyz="${-(length - strut_thickness)/2.0} ${-(width - strut_thickness)/2.0} 0" rpy="0 0 0"/>
+        <geometry>
+          <box size="${strut_thickness} ${strut_thickness} ${height}"/>
+        </geometry>
+      </visual>
+      <!-- Back Block -->
+      <visual>
+        <origin xyz="${-(length - 0.13)/2.0} 0 ${(height + 0.08)/2.0}" rpy="0 0 0"/>
+        <geometry>
+          <box size="0.13 0.4 0.08"/>
+        </geometry>
+      </visual>
+      <!-- Cylinder -->
+      <visual>
+        <origin xyz="${length/2.0 - 0.08 - 0.23/2.0} 0 ${0.11 + height/2.0}" rpy="0 ${pi/2} 0"/>
+        <geometry>
+          <cylinder radius="0.11" length="0.23"/>
         </geometry>
       </visual>

File: aquadrone_description/urdf/thruster.urdf.xacro (robot description, xacro)
@@ -4,7 +4,7 @@
     <link name="thruster_${thruster_id}">
       <visual>
-      <origin xyz="0.025 0 0" rpy="0 0 0"/>
+      <origin xyz="0 0 0" rpy="0 0 0"/>
         <geometry>
-          <box size="0.01 0.01 0.1"/>
+          <box size="0.06 0.01 0.08"/>
         </geometry>
       </visual>
@@ -12,5 +12,5 @@
         <origin xyz="0 0 0" rpy="0 ${pi/2} 0"/>
         <geometry>
-          <cylinder radius="0.01" length="0.05"/>
+          <cylinder radius="0.05" length="0.01"/>
         </geometry>
       </visual>

Commit message: change thruster angles to match real submarine

File: aquadrone_description/models/v28.urdf.xacro (robot description, xacro)
@@ -30,14 +30,14 @@
   <!-- UP/DOWN-->
   <xacro:thruster_macro thruster_id="0">
-    <origin xyz="0.2 0.285 0.1" rpy="0 ${pi/2} 0"/>
+    <origin xyz="0.2 0.285 0.1" rpy="0 ${-pi/2} 0"/>
   </xacro:thruster_macro>
   <xacro:thruster_macro thruster_id="1">
-    <origin xyz="0.2 -0.285 0.1" rpy="0 ${pi/2} 0"/>
+    <origin xyz="0.2 -0.285 0.1" rpy="0 ${-pi/2} 0"/>
   </xacro:thruster_macro>
   <xacro:thruster_macro thruster_id="2">
-    <origin xyz="-0.2 0.285 0.1" rpy="0 ${pi/2} 0"/>
+    <origin xyz="-0.2 0.285 0.1" rpy="0 ${-pi/2} 0"/>
   </xacro:thruster_macro>
   <xacro:thruster_macro thruster_id="3">
-    <origin xyz="-0.2 -0.285 0.1" rpy="0 ${pi/2} 0"/>
+    <origin xyz="-0.2 -0.285 0.1" rpy="0 ${-pi/2} 0"/>
   </xacro:thruster_macro>
 <!-- FORWARD/BACKWARD-->
@@ -50,5 +50,5 @@
 <!-- LEFT/RIGHT-->
 <xacro:thruster_macro thruster_id="6">
-    <origin xyz="0 0.17 0" rpy="0 0 ${-pi/2}"/>
+    <origin xyz="0 0.17 0" rpy="0 0 ${pi/2}"/>
   </xacro:thruster_macro>
    <xacro:thruster_macro thruster_id="7">

Commit message: thruster directions

File: aquadrone_description/models/v28.urdf.xacro (robot description, xacro)
@@ -50,5 +50,5 @@
 <!-- LEFT/RIGHT-->
 <xacro:thruster_macro thruster_id="6">
-    <origin xyz="0 0.17 0" rpy="0 0 ${-pi/2}"/>
+    <origin xyz="0 0.17 0" rpy="0 0 ${pi/2}"/>
   </xacro:thruster_macro>
    <xacro:thruster_macro thruster_id="7">

Commit message: clean up xacro file

File: aquadrone_description/models/v28.urdf.xacro (robot description, xacro)
@@ -1,57 +1,58 @@
 <?xml version="1.0"?>
-<robot name="aquadrone" xmlns:xacro="http://www.ros.org/wiki/xacro" >
-<!-- https://github.com/uuvsimulator/uuv_simulator/wiki/Templates-to-create-a-new-thruster-actuated-vehicle-model -->
-  <!-- Input debug flag -->
-  <xacro:arg name="debug" default="0"/>
+<robot name="aquadrone" xmlns:xacro="http://www.ros.org/wiki/xacro">
+    <!-- https://github.com/uuvsimulator/uuv_simulator/wiki/Templates-to-create-a-new-thruster-actuated-vehicle-model -->
+    <!-- Input debug flag -->
+    <xacro:arg name="debug" default="0"/>
     <xacro:property name="strut_thickness" value="0.02"/>
-  <!-- Describing the dimensions of the vehicle's bounding box -->
-  <xacro:property name="length" value="0.51"/>
-  <xacro:property name="width"  value="0.46"/>
-  <xacro:property name="height" value="0.2"/>
-  <!-- Include the ROV macro file -->
-  <xacro:include filename="$(find aquadrone_description)/urdf/aquadrone_v2.urdf.xacro"/>
-  <xacro:include filename="$(find aquadrone_description)/urdf/thruster.urdf.xacro"/>
-  <!-- Create the rov_example -->
-  <xacro:aquadrone_base debug="$(arg debug)" cog="0 0 0" cob="0 0 0"/>
+    <!-- Describing the dimensions of the vehicle's bounding box -->
+    <xacro:property name="length" value="0.51"/>
+    <xacro:property name="width" value="0.46"/>
+    <xacro:property name="height" value="0.2"/>
+    <!-- Include the ROV macro file -->
+    <xacro:include filename="$(find aquadrone_description)/urdf/aquadrone_v2.urdf.xacro"/>
+    <xacro:include filename="$(find aquadrone_description)/urdf/thruster.urdf.xacro"/>
+    <!-- Create the rov_example -->
+    <xacro:aquadrone_base debug="$(arg debug)" cog="0 0 0" cob="0 0 0"/>
     <!-- Pressure  -->
-  <xacro:include filename="$(find uuv_sensor_ros_plugins)/urdf/pressure_snippets.xacro"/>
-  <xacro:default_pressure namespace="aquadrone/out/" parent_link="base_link">
+    <xacro:include filename="$(find uuv_sensor_ros_plugins)/urdf/pressure_snippets.xacro"/>
+    <xacro:default_pressure namespace="aquadrone/out/" parent_link="base_link">
         <origin xyz="0 0 ${0.11 + 0.2/2.0}" rpy="0 ${pi/2.0} 0"/>
-  </xacro:default_pressure>
-  <!-- IMU -->
-  <xacro:include filename="$(find uuv_sensor_ros_plugins)/urdf/imu_snippets.xacro"/>
-  <xacro:default_imu namespace="aquadrone/out/" parent_link="base_link">
-    <origin xyz="0 0 0" rpy="0 0 0"/>
-  </xacro:default_imu>
-  <xacro:include filename="$(find aquadrone_description)/urdf/simple_camera.urdf.xacro"/>
-  <xacro:simple_camera_macro name="front_cam">
-    <origin xyz="${0.91/2.0 - 0.08 - 0.22/2.0} 0 ${0.11 + 0.2/2.0}" rpy="0 0 0"/>
-  </xacro:simple_camera_macro>
-  <!-- UP/DOWN-->
-  <xacro:thruster_macro thruster_id="0">
-    <origin xyz="0.2 0.285 0.1" rpy="0 ${pi/2} 0"/>
-  </xacro:thruster_macro>
-  <xacro:thruster_macro thruster_id="1">
-    <origin xyz="0.2 -0.285 0.1" rpy="0 ${pi/2} 0"/>
-  </xacro:thruster_macro>
-  <xacro:thruster_macro thruster_id="2">
-    <origin xyz="-0.2 0.285 0.1" rpy="0 ${pi/2} 0"/>
-  </xacro:thruster_macro>
-  <xacro:thruster_macro thruster_id="3">
-    <origin xyz="-0.2 -0.285 0.1" rpy="0 ${pi/2} 0"/>
-  </xacro:thruster_macro>
-<!-- FORWARD/BACKWARD-->
- <xacro:thruster_macro thruster_id="4">
-    <origin xyz="0 0.285 0.1" rpy="0 0 0"/>
-  </xacro:thruster_macro>
-   <xacro:thruster_macro thruster_id="5">
-    <origin xyz="0 -0.285 0.1" rpy="0 0 0"/>
-  </xacro:thruster_macro>
-<!-- LEFT/RIGHT-->
-<xacro:thruster_macro thruster_id="6">
-    <origin xyz="0 0.17 0" rpy="0 0 ${pi/2}"/>
-  </xacro:thruster_macro>
-   <xacro:thruster_macro thruster_id="7">
-    <origin xyz="0 -0.17 0" rpy="0 0 ${-pi/2}"/>
-  </xacro:thruster_macro>
+    </xacro:default_pressure>
+    <!-- IMU -->
+    <xacro:include filename="$(find uuv_sensor_ros_plugins)/urdf/imu_snippets.xacro"/>
+    <xacro:default_imu namespace="aquadrone/out/" parent_link="base_link">
+        <origin xyz="0 0 0" rpy="0 0 0"/>
+    </xacro:default_imu>
+    <!-- Camera -->
+    <xacro:include filename="$(find aquadrone_description)/urdf/simple_camera.urdf.xacro"/>
+    <xacro:simple_camera_macro name="front_cam">
+        <origin xyz="${0.91/2.0 - 0.08 - 0.22/2.0} 0 ${0.11 + 0.2/2.0}" rpy="0 0 0"/>
+    </xacro:simple_camera_macro>
+    <!-- UP/DOWN-->
+    <xacro:thruster_macro thruster_id="0">
+        <origin xyz="0.2 0.285 0.1" rpy="0 ${pi/2} 0"/>
+    </xacro:thruster_macro>
+    <xacro:thruster_macro thruster_id="1">
+        <origin xyz="0.2 -0.285 0.1" rpy="0 ${pi/2} 0"/>
+    </xacro:thruster_macro>
+    <xacro:thruster_macro thruster_id="2">
+        <origin xyz="-0.2 0.285 0.1" rpy="0 ${pi/2} 0"/>
+    </xacro:thruster_macro>
+    <xacro:thruster_macro thruster_id="3">
+        <origin xyz="-0.2 -0.285 0.1" rpy="0 ${pi/2} 0"/>
+    </xacro:thruster_macro>
+    <!-- FORWARD/BACKWARD-->
+    <xacro:thruster_macro thruster_id="4">
+        <origin xyz="0 0.285 0.1" rpy="0 0 0"/>
+    </xacro:thruster_macro>
+    <xacro:thruster_macro thruster_id="5">
+        <origin xyz="0 -0.285 0.1" rpy="0 0 0"/>
+    </xacro:thruster_macro>
+    <!-- LEFT/RIGHT-->
+    <xacro:thruster_macro thruster_id="6">
+        <origin xyz="0 0.17 0" rpy="0 0 ${pi/2}"/>
+    </xacro:thruster_macro>
+    <xacro:thruster_macro thruster_id="7">
+        <origin xyz="0 -0.17 0" rpy="0 0 ${-pi/2}"/>
+    </xacro:thruster_macro>
 </robot>
